Commit message: Make modular

File: tools/config/urdf/nandhi.urdf.xacro (robot description, xacro)
@@ -1,69 +1,5 @@
 <?xml version="1.0"?>
 <robot name="nandhi" xmlns:xacro="http://www.ros.org/wiki/xacro">
-    <xacro:property name="base_length" value="0.4" />
-    <xacro:property name="base_width" value="0.26" />
-    <xacro:property name="base_height" value="0.01" />
-    <xacro:property name="wheel_radius" value="0.045" />
-    <xacro:property name="wheel_length" value="0.04" />
-    <xacro:property name="wheel_link_pose" value="${(base_width / 2) + (wheel_length / 2)}"/>
-    <material name="green">
-        <color rgba="0 1 0 1" />
-    </material>
-    <material name="blue">
-        <color rgba="0 0 1 1" />
-    </material>
-    <link name="base_footprint" />
-    <link name="base_link">
-        <visual>
-            <geometry>
-                <box size="${base_length} ${base_width} ${base_height}" />
-            </geometry>
-            <origin xyz="0 0 ${base_height / 2}" rpy="0 0 0" />
-            <material name="blue" />
-        </visual>
-    </link>
-    <xacro:macro name="wheel_link" params="prefix">
-        <link name="${prefix}_wheel_link">
-            <visual>
-                <geometry>
-                    <cylinder radius="${wheel_radius}" length="${wheel_length}" />
-                </geometry>
-                <origin xyz="0 0 0" rpy="${pi / 2} 0 0" />
-                <material name="green" />
-            </visual>
-        </link>
-    </xacro:macro>
-    <xacro:wheel_link prefix="front_left" />
-    <xacro:wheel_link prefix="front_right" />
-    <xacro:wheel_link prefix="rear_left" />
-    <xacro:wheel_link prefix="rear_right" />
-    <joint name="base_joint" type="fixed">
-        <parent link="base_footprint" />
-        <child link="base_link" />
-        <origin xyz="0 0 ${wheel_radius}" rpy="0 0 0" />
-    </joint>
-    <joint name="base_front_left_wheel_joint" type="continuous">
-        <parent link="base_link" />
-        <child link="front_left_wheel_link" />
-        <origin xyz="-${wheel_link_pose} -${wheel_link_pose} ${base_height / 2}" rpy="0 0 0" />
-        <axis xyz="0 1 0" />
-    </joint>
-    <joint name="base_front_right_wheel_joint" type="continuous">
-        <parent link="base_link" />
-        <child link="front_right_wheel_link" />
-        <origin xyz="-${wheel_link_pose} ${wheel_link_pose} ${base_height / 2}" rpy="0 0 0" />
-        <axis xyz="0 1 0" />
-    </joint>
-    <joint name="base_rear_left_wheel_joint" type="continuous">
-        <parent link="base_link" />
-        <child link="rear_left_wheel_link" />
-        <origin xyz="${wheel_link_pose} -${wheel_link_pose} ${base_height / 2}" rpy="0 0 0" />
-        <axis xyz="0 1 0" />
-    </joint>
-    <joint name="base_rear_right_wheel_joint" type="continuous">
-        <parent link="base_link" />
-        <child link="rear_right_wheel_link" />
-        <origin xyz="${wheel_link_pose} ${wheel_link_pose} ${base_height / 2}" rpy="0 0 0" />
-        <axis xyz="0 1 0" />
-    </joint>
+    <xacro:include filename="common_properties.xacro" />
+    <xacro:include filename="robot_base.xacro" />
 </robot>
