Commit message: add collision and innertia

File: tools/config/urdf/common_properties.xacro (robot description, xacro)
@@ -7,3 +7,21 @@
         <color rgba="0 0 1 1" />
     </material>
+    <xacro:macro name="box_inertia" params="m l w h xyz rpy">
+        <inertial>
+            <origin xyz="${xyz}" rpy="${rpy}" />
+            <mass value="${m}" />
+            <inertia ixx="${(m/12) * (h*h + l*l)}" ixy="0" ixz="0"
+                iyy="${(m/12) * (w*w + l*l)}" iyz="0"
+                izz="${(m/12) * (w*w + h*h)}" />
+        </inertial>
+    </xacro:macro>
+    <xacro:macro name="cylinder_inertia" params="m r l xyz rpy">
+        <inertial>
+            <origin xyz="${xyz}" rpy="${rpy}" />
+            <mass value="${m}" />
+            <inertia ixx="${(m/12) * (3*r*r + l*l)}" ixy="0" ixz="0"
+                iyy="${(m/12) * (3*r*r + l*l)}" iyz="0"
+                izz="${(m/2) * (r*r)}" />
+        </inertial>
+    </xacro:macro>
 </robot>

File: tools/config/urdf/robot_base.xacro (robot description, xacro)
@@ -16,4 +16,12 @@
             <material name="blue" />
         </visual>
+        <collision>
+            <geometry>
+                <box size="${base_length} ${base_width} ${base_height}" />
+            </geometry>
+            <origin xyz="0 0 ${base_height / 2}" rpy="0 0 0" />
+        </collision>
+        <xacro:box_inertia m="3.0" l="${base_length}" w="${base_width}" h="${base_height}"
+            xyz="0 0 ${base_height / 2}" rpy="0 0 0" />
     </link>
     <xacro:macro name="wheel_link" params="prefix">
@@ -26,4 +34,12 @@
                 <material name="green" />
             </visual>
+            <collision>
+                <geometry>
+                    <cylinder radius="${wheel_radius}" length="${wheel_length}" />
+                </geometry>
+                <origin xyz="0 0 0" rpy="${pi / 2} 0 0" />
+            </collision>
+            <xacro:cylinder_inertia m="0.1" r="${wheel_radius}" l="${wheel_length}" xyz="0 0 0"
+                rpy="${pi / 2} 0 0" />
         </link>
     </xacro:macro>
@@ -43,4 +59,10 @@
         <axis xyz="0 1 0" />
     </joint>
+    <joint name="base_front_left_wheel_steer_joint" type="continuous">
+        <parent link="base_link" />
+        <child link="front_left_wheel_link" />
+        <origin xyz="-${wheel_link_pose} -${wheel_link_pose} ${base_height / 2}" rpy="0 0 0" />
+        <axis xyz="0 0 1" />
+    </joint>
     <joint name="base_front_right_wheel_joint" type="continuous">
         <parent link="base_link" />
@@ -48,4 +70,10 @@
         <origin xyz="-${wheel_link_pose} ${wheel_link_pose} ${base_height / 2}" rpy="0 0 0" />
         <axis xyz="0 1 0" />
+    </joint>
+    <joint name="base_front_right_wheel_steer_joint" type="continuous">
+        <parent link="base_link" />
+        <child link="front_right_wheel_link" />
+        <origin xyz="-${wheel_link_pose} ${wheel_link_pose} ${base_height / 2}" rpy="0 0 0" />
+        <axis xyz="0 0 1" />
     </joint>
     <joint name="base_rear_left_wheel_joint" type="continuous">

Commit message: Minor Fix for on the fly xacro to urdf

File: tools/config/urdf/common_properties.xacro (robot description, xacro)
@@ -6,4 +6,22 @@
     <material name="blue">
         <color rgba="0 0 1 1" />
+    </material>
+    <material name="green">
+        <color rgba="0.0 0.8 0.0 1.0" />
+    </material>
+    <material name="grey">
+        <color rgba="0.2 0.2 0.2 1.0" />
+    </material>
+    <material name="orange">
+        <color rgba="${255/255} ${108/255} ${10/255} 1.0" />
+    </material>
+    <material name="brown">
+        <color rgba="${222/255} ${207/255} ${195/255} 1.0" />
+    </material>
+    <material name="red">
+        <color rgba="0.8 0.0 0.0 1.0" />
+    </material>
+    <material name="white">
+        <color rgba="1.0 1.0 1.0 1.0" />
     </material>
     <xacro:macro name="box_inertia" params="m l w h xyz rpy">

Commit message: add world and rename base_link to chassis

File: tools/config/urdf/common_properties.xacro (robot description, xacro)
@@ -6,7 +6,4 @@
     <material name="blue">
         <color rgba="0 0 1 1" />
-    </material>
-    <material name="green">
-        <color rgba="0.0 0.8 0.0 1.0" />
     </material>
     <material name="grey">
@@ -27,5 +24,5 @@
     <xacro:macro name="box_inertia" params="m l w h xyz rpy">
         <inertial>
-            <origin xyz="${xyz}" rpy="${rpy}" />
+            <origin rpy="${rpy}" xyz="${xyz}"/>
             <mass value="${m}" />
             <inertia ixx="${(m/12) * (h*h + l*l)}" ixy="0" ixz="0"
@@ -36,5 +33,5 @@
     <xacro:macro name="cylinder_inertia" params="m r l xyz rpy">
         <inertial>
-            <origin xyz="${xyz}" rpy="${rpy}" />
+            <origin rpy="${rpy}" xyz="${xyz}"/>
             <mass value="${m}" />
             <inertia ixx="${(m/12) * (3*r*r + l*l)}" ixy="0" ixz="0"

File: tools/config/urdf/robot_base.xacro (robot description, xacro)
@@ -7,8 +7,11 @@
     <xacro:property name="wheel_length" value="0.04" />
     <xacro:property name="wheel_link_pose" value="${(base_width / 2) + (wheel_length / 2)}" />
-    <link name="base_footprint" />
-    <link name="base_link">
+    <link name="base_link" />
+    <link name="chassis">
+        <xacro:box_inertia m="3.0" l="${base_length}" w="${base_width}" h="${base_height}"
+        xyz="0 0 ${base_height / 2}" rpy="0 0 0" />
         <visual>
             <geometry>
+                <!-- <mesh filename="chassis.STL" /> -->
                 <box size="${base_length} ${base_width} ${base_height}" />
             </geometry>
@@ -22,9 +25,9 @@
             <origin xyz="0 0 ${base_height / 2}" rpy="0 0 0" />
         </collision>
-        <xacro:box_inertia m="3.0" l="${base_length}" w="${base_width}" h="${base_height}"
-            xyz="0 0 ${base_height / 2}" rpy="0 0 0" />
     </link>
     <xacro:macro name="wheel_link" params="prefix">
         <link name="${prefix}_wheel_link">
+            <xacro:cylinder_inertia m="0.1" r="${wheel_radius}" l="${wheel_length}" xyz="0 0 0"
+            rpy="${pi / 2} 0 0" />
             <visual>
                 <geometry>
@@ -32,5 +35,5 @@
                 </geometry>
                 <origin xyz="0 0 0" rpy="${pi / 2} 0 0" />
-                <material name="green" />
+                <material name="grey" />
             </visual>
             <collision>
@@ -40,6 +43,4 @@
                 <origin xyz="0 0 0" rpy="${pi / 2} 0 0" />
             </collision>
-            <xacro:cylinder_inertia m="0.1" r="${wheel_radius}" l="${wheel_length}" xyz="0 0 0"
-                rpy="${pi / 2} 0 0" />
         </link>
     </xacro:macro>
@@ -49,10 +50,10 @@
     <xacro:wheel_link prefix="rear_right" />
     <joint name="base_joint" type="fixed">
-        <parent link="base_footprint" />
-        <child link="base_link" />
+        <parent link="base_link" />
+        <child link="chassis" />
         <origin xyz="0 0 ${wheel_radius}" rpy="0 0 0" />
     </joint>
     <joint name="base_front_left_wheel_joint" type="continuous">
-        <parent link="base_link" />
+        <parent link="chassis" />
         <child link="front_left_wheel_link" />
         <origin xyz="-${wheel_link_pose} -${wheel_link_pose} ${base_height / 2}" rpy="0 0 0" />
@@ -60,5 +61,5 @@
     </joint>
     <joint name="base_front_right_wheel_joint" type="continuous">
-        <parent link="base_link" />
+        <parent link="chassis" />
         <child link="front_right_wheel_link" />
         <origin xyz="-${wheel_link_pose} ${wheel_link_pose} ${base_height / 2}" rpy="0 0 0" />
@@ -66,5 +67,5 @@
     </joint>
     <joint name="base_rear_left_wheel_joint" type="continuous">
-        <parent link="base_link" />
+        <parent link="chassis" />
         <child link="rear_left_wheel_link" />
         <origin xyz="${wheel_link_pose} -${wheel_link_pose} ${base_height / 2}" rpy="0 0 0" />
@@ -72,5 +73,5 @@
     </joint>
     <joint name="base_rear_right_wheel_joint" type="continuous">
-        <parent link="base_link" />
+        <parent link="chassis" />
         <child link="rear_right_wheel_link" />
         <origin xyz="${wheel_link_pose} ${wheel_link_pose} ${base_height / 2}" rpy="0 0 0" />
